File: PCM9211.kicad_sch (KiCad schematic)
At the start: 48 parts, among them J12 3.5mm Jack, J3 RCJ-041, J4 HDMI Port, J5 Optical Jack, T1 2.06mH, U2 PCM9211PTR, U5 USBLC6-4SC6-EV

Commit message: Remove AGND
Connections:
- net AGND is gone; now on net GND: C38.2, C39.2, C42.2, C43.2, D3.3 (common), J12.RN, J12.S, R24.2, R25.2, U2.41 (AGND)
