File: TAS3251.kicad_sch (KiCad schematic)
At the start: 57 parts, among them J1 1715721, J2 1715721, U1 TAS3251DKQR

Commit message: Remove AGND
Connections:
- net AGND is gone; now on net GND: C10.2, C9.2, U1.55 (AGND)
