File: FSC_BT1026E.kicad_sch (KiCad schematic)
At the start: 6 parts, among them U3 FCS-BT1026E

Commit message: Add TP1,2 for I2C. Add 0 ohm for 5V to BT module
Parts:
- added R38: 0, symbol Device:R_US
Connections:
- net 5V: now also R38.1; no longer U3.39 (VCC_CHG)
- new net: R38.2, U3.39 (VCC_CHG)
Other:
- note added: "0603 or 0805 No-pop by default seems like I won't need it"
Changed lines of the file:
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@@
 	(text "This will be the pinout unless I find out it donesn't work \nand I have to use I2S"
 		(exclude_from_sim no)
-		(at 156.718 49.53 0)
+		(at 156.464 51.308 0)
 		(effects
 			(font
 				(size 1.27 1.27)
 			)
+		)
+	)
+	(text "0603 or 0805\nNo-pop by default seems like I won't need it"
+		(exclude_from_sim no)
+		(at 127.508 39.878 0)
+		(effects
+			(font
+				(size 1.27 1.27)
+			)
+			(justify left)
 		)
 	)
@@
 	(wire
 		(pts
+			(xy 120.65 44.45) (xy 120.65 63.5)
+		)
+		(stroke
+			(width 0)
+			(type default)
+		)
+	)
+	(wire
+		(pts
 			(xy 171.45 142.24) (xy 171.45 144.78)
 		)
@@
 	(wire
 		(pts
-			(xy 120.65 35.56) (xy 120.65 63.5)
-		)
-		(stroke
-			(width 0)
-			(type default)
-		)
-	)
-	(wire
-		(pts
 			(xy 120.65 63.5) (xy 121.92 63.5)
 		)
@@
 		(pts
 			(xy 170.18 139.7) (xy 171.45 139.7)
+		)
+		(stroke
+			(width 0)
+			(type default)
+		)
+	)
+	(wire
+		(pts
+			(xy 120.65 35.56) (xy 120.65 36.83)
 		)
 		(stroke
@@
 					(unit 1)
 				)
+			)
+		)
+	)
+	(symbol
+		(lib_id "Device:R_US")
+		(at 120.65 40.64 0)
+		(unit 1)
+		(body_style 1)
+		(exclude_from_sim no)
+		(in_bom yes)
+		(on_board yes)
+		(in_pos_files yes)
+		(dnp yes)
+		(fields_autoplaced yes)
+		(property "Reference" "R38"
+			(at 123.19 39.3699 0)
+			(show_name no)
+			(do_not_autoplace no)
+			(effects
+				(font
+					(size 1.27 1.27)
+				)
+				(justify left)
+			)
+		)
+		(property "Value" "0"
+			(at 123.19 41.9099 0)
+			(show_name no)
+			(do_not_autoplace no)
+			(effects
+				(font
+					(size 1.27 1.27)
+				)
+				(justify left)
+			)
+		)
+		(property "Footprint" ""
+			(at 121.666 40.894 90)
+			(hide yes)
+			(show_name no)
+			(do_not_autoplace no)
+			(effects
+				(font
+					(size 1.27 1.27)
+				)
+			)
+		)
+		(property "Datasheet" ""
+			(at 120.65 40.64 0)
+			(hide yes)
+			(show_name no)
+			(do_not_autoplace no)
+			(effects
+				(font
+					(size 1.27 1.27)
+				)
+			)
+		)
+		(property "Description" "Resistor, US symbol"
+			(at 120.65 40.64 0)
+			(hide yes)
+			(show_name no)
+			(do_not_autoplace no)
+			(effects
+				(font
+					(size 1.27 1.27)
+				)
+			)
+		)
+		(pin "2"
+		)
+		(pin "1"
+		)
+		(instances
+			(project "Blamp"
+				(path "/90f900ff-e6f7-4b42-9414-7e4ea0d3c559/841b646d-11f9-48f0-98ae-69b9b8752b35"
+					(reference "R38")
+					(unit 1)
+				)
